Commit message: change BicycleSteeringController

File: trxbewi_control/xacro/mobile_base.ros2_control.xacro (robot description, xacro)
@@ -15,14 +15,17 @@
                 </xacro:unless>
             </hardware>
-            <joint name="thottle">
+            <joint name="virtual_throttle_joint">
                 <command_interface name="velocity"/>
                 <state_interface name="velocity"/>
+                <state_interface name="position"/>
                 <param name="max_rpm">2500</param>
             </joint>
-            <joint name="steering">
+            <joint name="virtual_steering_joint">
                 <command_interface name="position"/>
                 <state_interface name="position"/>
+                <state_interface name="velocity"/>
                 <param name="max_degrees">180</param>
             </joint>
+            <!--
             <joint name="gear">
                 <command_interface name="position"/>
@@ -40,4 +43,5 @@
                 <param name="max_degrees">180</param>
             </joint>
+            -->
         </ros2_control>
     </xacro:macro>

File: trxbewi_description/urdf/common_properties.xacro (robot description, xacro)
@@ -25,4 +25,7 @@
     <material name="red">
         <color rgba="1 0 0 1" />
+    </material>
+    <material name="invisible">
+        <color rgba="0.0 0.0 0.0 0.0"/>
     </material>
     <xacro:macro name="box_inertia" params="m l w h xyz rpy">

File: trxbewi_description/urdf/mobile_base.xacro (robot description, xacro)
@@ -32,5 +32,5 @@
             </inertial>
         </link>
-        <joint name="${name}_axle_joint" type="revolute">
+        <joint name="${name}_axle_joint" type="fixed">
             <parent link="base_link" />
             <child link="${name}_axle_link" />
@@ -38,19 +38,8 @@
             <axis xyz="1 0 0" />
             <limit effort="10.0" lower="-0.5" upper="0.5" velocity="1.0" />
+            <dynamics damping="0.2"/>
         </joint>
     </xacro:macro>
     <xacro:macro name="spindle" params="name radius length mass color origin_x origin_y origin_z">
-        <xacro:if value="${name == 'left_front'}">
-            <xacro:property name="position" value="front" />
-        </xacro:if>
-        <xacro:if value="${name == 'right_front'}">
-            <xacro:property name="position" value="front" />
-        </xacro:if>
-        <xacro:if value="${name == 'left_rear'}">
-            <xacro:property name="position" value="rear" />
-        </xacro:if>
-        <xacro:if value="${name == 'right_rear'}">
-            <xacro:property name="position" value="rear" />
-        </xacro:if>
         <link name="${name}_spindle_link">
             <visual>
@@ -73,13 +62,26 @@
             </inertial>
         </link>
-        <joint name="${name}_steering_joint" type="revolute">
-            <parent link="${position}_axle_link" />
+        <joint name="${name}_steering_joint" type="fixed">
+            <parent link="front_axle_link" />
             <child link="${name}_spindle_link" />
             <origin xyz="${origin_x} ${origin_y} ${origin_z}" rpy="0 0 0" />
             <axis xyz="0 0 1" />
             <limit effort="10.0" lower="-0.5" upper="0.5" velocity="1.0" />
+            <!--<mimic joint="virtual_steering_joint" multiplier="1.0" offset="0.0"/>-->
         </joint>
     </xacro:macro>
     <xacro:macro name="wheel" params="name radius length mass color origin_x origin_y origin_z">
+        <xacro:if value="${name == 'left_front'}">
+            <xacro:property name="position" value="front" />
+        </xacro:if>
+        <xacro:if value="${name == 'right_front'}">
+            <xacro:property name="position" value="front" />
+        </xacro:if>
+        <xacro:if value="${name == 'left_rear'}">
+            <xacro:property name="position" value="rear" />
+        </xacro:if>
+        <xacro:if value="${name == 'right_rear'}">
+            <xacro:property name="position" value="rear" />
+        </xacro:if>
         <link name="${name}_wheel_link">
             <visual>
@@ -102,5 +104,6 @@
             </inertial>
         </link>
-        <joint name="${name}_rotation_joint" type="continuous">
+        <xacro:if value="${position == 'front'}">
+        <joint name="${name}_rotation_joint" type="fixed">
             <parent link="${name}_spindle_link" />
             <child link="${name}_wheel_link" />
@@ -108,12 +111,20 @@
             <axis xyz="0 1 0" />
         </joint>
-        <!-- Joint prismatic pour la suspension -->
+        </xacro:if>
+        <xacro:if value="${position == 'rear'}">
+        <joint name="${name}_rotation_joint" type="fixed">
+            <parent link="virtual_throttle" />
+            <child link="${name}_wheel_link" />
+            <origin xyz="${origin_x} ${origin_y} ${origin_z}" rpy="0 0 0" />
+        </joint>
+        </xacro:if>
+        <!-- Joint prismatic pour la suspension
         <joint name="${name}_suspension_joint" type="prismatic">
             <parent link="${name}_spindle_link" />
             <child link="${name}_wheel_link" />
             <origin xyz="0 0 0" rpy="0 0 0" />
-            <axis xyz="0 0 1" /> <!-- Mouvement vertical de la suspension -->
-            <limit lower="0" upper="0.02" effort="100.0" velocity="1.0" /> <!-- Course de 2 cm -->
-        </joint>
+            <axis xyz="0 0 1" />
+            <limit lower="0" upper="0.02" effort="100.0" velocity="1.0" />
+        </joint> -->
     </xacro:macro>
     <!-- Châssis principal -->
@@ -145,13 +156,55 @@
         <axis xyz="0 0 0" />
     </joint>
+    <link name="virtual_steering">
+        <visual>
+            <origin xyz="0 0 0" rpy="${pi / 2} 0 0"/>
+            <geometry>
+                <cylinder length="0.01" radius="${wheel_radius}"/>
+            </geometry>
+            <material name="black"/>
+        </visual>
+        <inertial>
+            <mass value="0.001"/>
+            <origin xyz="0 0 0"/>
+            <inertia ixx="0.001" ixy="0" ixz="0" iyy="0.001" iyz="0" izz="0.001"/>
+        </inertial>
+    </link>
+    <joint name="virtual_steering_joint" type="revolute">
+        <parent link="front_axle_link"/>
+        <child link="virtual_steering"/>
+        <origin xyz="0 0 0" rpy="0 0 0"/>
+        <axis xyz="0 0 1"/>
+        <limit lower="-0.4" upper="0.4" effort="10.0" velocity="0.0"/>
+        <dynamics damping="0.2"/>
+    </joint>
+    <link name="virtual_throttle">
+        <visual>
+            <origin xyz="0 0 0" rpy="${pi / 2} 0 0"/>
+            <geometry>
+                <cylinder length="0.01" radius="${wheel_radius}"/>
+            </geometry>
+            <material name="black"/>
+        </visual>
+        <inertial>
+            <mass value="0.001"/>
+            <origin xyz="0 0 0"/>
+            <inertia ixx="0.001" ixy="0" ixz="0" iyy="0.001" iyz="0" izz="0.001"/>
+        </inertial>
+    </link>
+    <joint name="virtual_throttle_joint" type="continuous">
+        <parent link="rear_axle_link"/>
+        <child link="virtual_throttle"/>
+        <origin xyz="0 0 0" rpy="0 0 0"/>
+        <axis xyz="0 1 0"/>
+        <limit effort="10.0" velocity="10.0"/>
+        <dynamics damping="0.2"/>
+    </joint>
     <xacro:axle name="front" radius="0.03" length="0.25" mass="1.0" color="black" origin_x="${wheelbase / 2}" origin_y="0" origin_z="0" />
     <xacro:axle name="rear" radius="0.03" length="0.25" mass="1.0" color="black" origin_x="-${wheelbase / 2}" origin_y="0" origin_z="0" />
     <xacro:spindle name="right_front" radius="0.015" length="0.04" mass="0.2" color="grey" origin_x="0" origin_y="${axle_length / 2}"  origin_z="0" />
     <xacro:spindle name="left_front" radius="0.015" length="0.04" mass="0.2" color="grey" origin_x="0" origin_y="-${axle_length / 2}"  origin_z="0" />
-    <xacro:spindle name="right_rear" radius="0.015" length="0.04" mass="0.2" color="grey" origin_x="0" origin_y="${axle_length / 2}"  origin_z="0" />
-    <xacro:spindle name="left_rear" radius="0.015" length="0.04" mass="0.2" color="grey" origin_x="0" origin_y="-${axle_length / 2}"  origin_z="0" />
     <xacro:wheel name="right_front" radius="${wheel_radius}" length="${wheel_length}" mass="0.5" color="black" origin_x="0" origin_y="0" origin_z="0" />
     <xacro:wheel name="left_front" radius="${wheel_radius}" length="${wheel_length}" mass="0.5" color="black" origin_x="0" origin_y="0" origin_z="0" />
-    <xacro:wheel name="right_rear" radius="${wheel_radius}" length="${wheel_length}" mass="0.5" color="black" origin_x="0" origin_y="0" origin_z="0" />
-    <xacro:wheel name="left_rear" radius="${wheel_radius}" length="${wheel_length}" mass="0.5" color="black" origin_x="0" origin_y="0" origin_z="0" />
+    <xacro:wheel name="right_rear" radius="${wheel_radius}" length="${wheel_length}" mass="0.5" color="black" origin_x="0" origin_y="${axle_length / 2}" origin_z="0" />
+    <xacro:wheel name="left_rear" radius="${wheel_radius}" length="${wheel_length}" mass="0.5" color="black" origin_x="0" origin_y="-${axle_length / 2}" origin_z="0" />
 </robot>
