Commit message: add cmd

File: shared/trxbewi_description/urdf/trx4_base.xacro (robot description, xacro)
@@ -66,4 +66,34 @@
     </inertial>
   </link>
+  <!-- CMD -->
+    <link name="steering_cmd">
+      <visual>
+        <geometry><cylinder length="0.02" radius="0.01"/></geometry>
+        <material name="metal"><color rgba="${mat_color}"/></material>
+      </visual>
+    </link>
+    <joint name="steering_cmd_joint" type="revolute">
+      <parent link="chassis"/>
+      <child  link="steering_cmd"/>
+      <origin xyz="0.16 0 0.06" rpy="0 0 0"/>
+      <axis xyz="0 0 1"/>
+      <limit lower="${radians(-35)}" upper="${radians(35)}" effort="800" velocity="${radians(180)}"/>
+      <dynamics damping="5.0" friction="0.2"/>
+    </joint>
+    <link name="traction_cmd">
+      <visual>
+        <origin xyz="0.0 0 0.0" rpy="${radians(90)} 0 0"/>
+        <geometry><cylinder length="0.06" radius="0.02"/></geometry>
+        <material name="metal"><color rgba="${mat_color}"/></material>
+      </visual>
+    </link>
+    <joint name="traction_cmd_joint" type="continuous">
+      <parent link="chassis"/>
+      <child  link="traction_cmd"/>
+      <origin xyz="0.08 0 0.03" rpy="0 0 ${radians(90)}"/>
+      <axis xyz="0 1 0"/>
+      <limit lower="${radians(-35)}" upper="${radians(35)}" effort="800" velocity="${radians(180)}"/>
+      <dynamics damping="5.0" friction="0.2"/>
+    </joint>
   <!-- ===== GÉNÉRATEUR ROUE+PORTE-MOYEU AV/ARR =====
       params:
@@ -118,4 +148,5 @@
         <limit lower="${radians(-35)}" upper="${radians(35)}" effort="800" velocity="${radians(180)}"/>
         <dynamics damping="5.0" friction="0.2"/>
+        <mimic joint="steering_cmd_joint" multiplier="1.0" offset="0.0"/>
       </joint>
     </xacro:if>
@@ -154,4 +185,5 @@
       <axis xyz="0 1 0"/>
       <dynamics damping="0.01" friction="0.05"/>
+      <mimic joint="traction_cmd_joint" multiplier="1.0" offset="0.0"/>
     </joint>
   </xacro:macro>

File: shared/trxbewi_description/urdf/trxbewi.urdf.xacro (robot description, xacro)
@@ -33,3 +33,7 @@
     xyz="0 0 0" rpy="0 0 0" />
   </link>
+  <joint name="$trxbewi_joint" type="fixed">
+    <parent link="base_link" />
+    <child link="chassis" />
+  </joint>
 </robot>

Commit message: _susp_joint fixed

File: shared/trxbewi_description/urdf/trx4_base.xacro (robot description, xacro)
@@ -119,5 +119,6 @@
       </collision>
     </link>
-    <joint name="${side}_susp_joint" type="prismatic">
+    <!-- <joint name="${side}_susp_joint" type="prismatic"> -->
+    <joint name="${side}_susp_joint" type="fixed">
       <parent link="chassis"/>
       <child  link="${side}_susp_link"/>
