Commit message: refact mobile base

File: core/trxbewi_control/xacro/mobile_base.ros2_control.xacro (robot description, xacro)
@@ -15,5 +15,5 @@
                 </xacro:unless>
             </hardware>
-            <joint name="virtual_throttle_joint">
+             <joint name="traction_cmd_joint">
                 <command_interface name="velocity"/>
                 <param name="port_id">0</param>
@@ -22,5 +22,5 @@
                 <param name="max_rpm">2500</param>
             </joint>
-            <joint name="virtual_steering_joint">
+            <joint name="steering_cmd_joint">
                 <command_interface name="position"/>
                 <param name="port_id">1</param>

File: shared/trxbewi_description/urdf/trxbewi.urdf.xacro (robot description, xacro)
@@ -7,5 +7,5 @@
   <xacro:include filename="$(find trxbewi_description)/urdf/common_properties.xacro" />
   <!-- Import trxbewi mobile base -->
-  <xacro:include filename="$(find trxbewi_description)/urdf/mobile_base.xacro" />
+  <xacro:include filename="$(find trxbewi_description)/urdf/trx4_base.xacro" />
   <!-- Import Sensors
   <xacro:include filename="$(find trxbewi_description)/urdf/sensors.xacro" />
